Commit message: Modified xacro file to include visual elements. Added move_turtle node and launchfile to test motion of turtle robot. Added waypoint_turtle node and launchfile to test waypoint motion control of turtle robot.

File: turtle_brick/urdf/turtle.urdf.xacro (robot description, xacro)
@@ -1,5 +1,5 @@
 <robot name="turtle" xmlns:xacro="http://wiki.ros.org/wiki/xacro">
-  <!-- slidebot is a robot that has 1 linear and 1 rotational degree of freedom -->
-  <!-- The base from which the body slides -->
+  <!-- turtlebot is a robot that has 3 rotational degree of freedom of which 2 are continuous-->
+  <!-- Functional parameters -->
   <xacro:property name="scale" value="0.4" />
   <xacro:property name="golden" value="1.618" />
@@ -10,8 +10,18 @@
   <xacro:property name="stem_length" value="${wheel_thickness / golden}" />
   <xacro:property name="stem_radius" value="${0.5 * wheel_thickness / (golden * golden)}" />
-  <xacro:property name="platform_radius" value="${0.5 * body_width * golden}" />
+  <xacro:property name="platform_radius" value="${0.85 * 0.5 * body_width * golden}" />
   <xacro:property name="pole_length" value="${body_height * (golden - 1) / golden}" />
   <xacro:property name="platform_thickness" value="${pole_length * (golden - 1)}" />
   <xacro:property name="pole_radius" value="${platform_thickness * golden}" />
+  <!-- Visual turtle elements-->
+  <xacro:property name="head_radius" value="${body_width * (golden - 1)/2}" />
+  <xacro:property name="head_offset" value="${1.1 * head_radius / golden}" />
+  <xacro:property name="foot_radius" value="${body_width * (golden - 1)/ (golden * 2)}" />
+  <xacro:property name="foot_offset_front" value="${foot_radius / (2 * golden)}" />
+  <xacro:property name="foot_offset_side" value="${foot_radius / (2 * golden)}" />
+  <xacro:property name="foot_height" value="${foot_radius / golden}" />
+  <xacro:property name="tail_length" value="${body_height/golden}" />
+  <xacro:property name="tail_width" value="${tail_length/golden}" />
+  <xacro:property name="tail_height" value="${tail_width/golden}" />
   <link name="base_link">
     <visual>
@@ -21,5 +31,5 @@
       </geometry>
       <material name="base_mat">
-        <color rgba="0 1 0 0.99" />
+        <color rgba="0.4 0.15 0 1" />
       </material>
     </visual>
@@ -42,15 +52,14 @@
       </material>
     </visual>
-    <collision>
+    <!-- <collision>
       <origin xyz="0 0 ${-stem_length/2}" rpy="0 0 0" />
       <geometry>
         <cylinder radius="${stem_radius}" length="${stem_length}" />
       </geometry>
-    </collision>
-  </link>
-  <joint name="swivel" type="revolute">
+    </collision> -->
+  </link>
+  <joint name="swivel" type="continuous">
     <origin xyz="0 0 ${-body_height/2}" rpy="0 0 0" />
     <axis xyz="0 0 1"/>
-    <limit lower="${-pi}" upper="${pi}" effort="100.0" velocity="100.0"/>
     <parent link="base_link" />
     <child link="stem" />
@@ -63,5 +72,5 @@
       </geometry>
       <material name="wheel_mat">
-        <color rgba="0.1 0.1 0.1 1" />
+        <color rgba="1 1 1 1" />
       </material>
     </visual>
@@ -74,5 +83,5 @@
   </link>
   <joint name="wheel_axle" type="continuous">
-    <origin xyz="0 0 ${-stem_length/2 - wheel_radius}" rpy="${pi/2} 0 0" />
+    <origin xyz="0 0 ${-stem_length/2 - wheel_radius}" rpy="${-pi/2} 0 0" />
     <axis xyz="0 0 1"/>
     <parent link="stem" />
@@ -108,5 +117,5 @@
       </geometry>
       <material name="platform_mat">
-        <color rgba="0.6 0.7 0 1" />
+        <color rgba="0.8 0.3 0 1" />
       </material>
     </visual>
@@ -121,7 +130,104 @@
     <origin xyz="0 0 ${pole_length/2}" rpy="0 0 0" />
     <axis xyz="0 1 0"/>
-    <limit lower="${-pi}" upper="${pi}" effort="100.0" velocity="100.0"/>
+    <limit lower="${-0.187}" upper="${0.187}" effort="100.0" velocity="100.0"/>
     <parent link="pole" />
     <child link="platform" />
   </joint>
+  <!-- Fixed visual elements-->
+  <link name="head">
+    <visual>
+      <origin xyz="${head_offset} 0 0" rpy="0 0 0" />
+      <geometry>
+        <sphere radius="${head_radius}" />
+      </geometry>
+      <material name="head_mat">
+        <color rgba="0.1 1 0 1" />
+      </material>
+    </visual>
+  </link>
+  <joint name="base2head" type="fixed">
+    <origin xyz="${body_width/2} 0 0" rpy="0 0 0" />
+    <parent link="base_link" />
+    <child link="head" />
+  </joint>
+  <link name="FL_leg">
+    <visual>
+      <origin xyz="${foot_offset_front} ${foot_offset_side} 0" rpy="0 0 0" />
+      <geometry>
+        <cylinder radius="${foot_radius}" length="${foot_height}"/>
+      </geometry>
+      <material name="head_mat">
+        <color rgba="0.1 1 0 1" />
+      </material>
+    </visual>
+  </link>
+  <joint name="base2FL" type="fixed">
+    <origin xyz="${body_width/2} ${body_width/2} ${-body_height/2 + foot_height/2}" rpy="0 0 0" />
+    <parent link="base_link" />
+    <child link="FL_leg" />
+  </joint>
+  <link name="FR_leg">
+    <visual>
+      <origin xyz="${foot_offset_front} ${-foot_offset_side} 0" rpy="0 0 0" />
+      <geometry>
+        <cylinder radius="${foot_radius}" length="${foot_height}"/>
+      </geometry>
+      <material name="head_mat">
+        <color rgba="0.1 1 0 1" />
+      </material>
+    </visual>
+  </link>
+  <joint name="base2FR" type="fixed">
+    <origin xyz="${body_width/2} ${-body_width/2} ${-body_height/2 + foot_height/2}" rpy="0 0 0" />
+    <parent link="base_link" />
+    <child link="FR_leg" />
+  </joint>
+  <link name="BL_leg">
+    <visual>
+      <origin xyz="${-foot_offset_front} ${foot_offset_side} 0" rpy="0 0 0" />
+      <geometry>
+        <cylinder radius="${foot_radius}" length="${foot_height}"/>
+      </geometry>
+      <material name="head_mat">
+        <color rgba="0.1 1 0 1" />
+      </material>
+    </visual>
+  </link>
+  <joint name="base2BL" type="fixed">
+    <origin xyz="${-body_width/2} ${body_width/2} ${-body_height/2 + foot_height/2}" rpy="0 0 0" />
+    <parent link="base_link" />
+    <child link="BL_leg" />
+  </joint>
+  <link name="BR_leg">
+    <visual>
+      <origin xyz="${-foot_offset_front} ${-foot_offset_side} 0" rpy="0 0 0" />
+      <geometry>
+        <cylinder radius="${foot_radius}" length="${foot_height}"/>
+      </geometry>
+      <material name="head_mat">
+        <color rgba="0.1 1 0 1" />
+      </material>
+    </visual>
+  </link>
+  <joint name="base2BR" type="fixed">
+    <origin xyz="${-body_width/2} ${-body_width/2} ${-body_height/2 + foot_height/2}" rpy="0 0 0" />
+    <parent link="base_link" />
+    <child link="BR_leg" />
+  </joint>
+  <link name="tail">
+    <visual>
+      <origin xyz="${-tail_length/2} 0 0" rpy="0 0 0" />
+      <geometry>
+        <box size="${tail_length} ${tail_width} ${tail_height}"/>
+      </geometry>
+      <material name="head_mat">
+        <color rgba="0.1 1 0 1" />
+      </material>
+    </visual>
+  </link>
+  <joint name="base2tail" type="fixed">
+    <origin xyz="${-body_width/2} 0 ${-tail_height/2}" rpy="0 0 0" />
+    <parent link="base_link" />
+    <child link="tail" />
+  </joint>
 </robot>

Commit message: Created message tyoe Tilt.msg in turtle_brick_interfaces. Created first draft of run_turtle.py node and run_turtle_launch.xml.

File: turtle_brick/urdf/turtle.urdf.xacro (robot description, xacro)
@@ -112,5 +112,5 @@
   <link name="platform">
     <visual>
-      <origin xyz="0 0 ${platform_thickness/2}" rpy="0 0 0" />
+      <origin xyz="0 0 0" rpy="0 0 0" />
       <geometry>
         <cylinder radius="${platform_radius}" length="${platform_thickness}" />
@@ -128,5 +128,5 @@
   </link>
   <joint name="tip" type="revolute">
-    <origin xyz="0 0 ${pole_length/2}" rpy="0 0 0" />
+    <origin xyz="0 0 ${pole_length/2 + platform_thickness/2}" rpy="0 0 0" />
     <axis xyz="0 1 0"/>
     <limit lower="${-0.187}" upper="${0.187}" effort="100.0" velocity="100.0"/>

Commit message: Added turtle.yaml configuration file. Added brick sliding off the platform behaviour.

File: turtle_brick/urdf/turtle.urdf.xacro (robot description, xacro)
@@ -1,12 +1,16 @@
 <robot name="turtle" xmlns:xacro="http://wiki.ros.org/wiki/xacro">
   <!-- turtlebot is a robot that has 3 rotational degree of freedom of which 2 are continuous-->
+  <xacro:property name="turtle_params" value="$(find turtle_brick)/turtle.yaml" />
+  <xacro:property name="params" value="${xacro.load_yaml(turtle_params)['/**']['ros__parameters']}" />
+  <xacro:property name="PLATFORM_HEIGHT" value="${params['platform_height']}" />
+  <xacro:property name="WHEEL_RADIUS" value="${params['wheel_radius']}" />
   <!-- Functional parameters -->
   <xacro:property name="scale" value="0.4" />
   <xacro:property name="golden" value="1.618" />
   <xacro:property name="wheel_thickness" value="${scale / golden}" />
-  <xacro:property name="wheel_radius" value="${golden * wheel_thickness / 2}" />
+  <xacro:property name="wheel_radius" value="${WHEEL_RADIUS}" />
   <xacro:property name="body_width" value="${golden * scale}" />
   <xacro:property name="body_height" value="${body_width / golden}" />
-  <xacro:property name="stem_length" value="${wheel_thickness / golden}" />
+  <!-- <xacro:property name="stem_length" value="${wheel_thickness / golden}" /> -->
   <xacro:property name="stem_radius" value="${0.5 * wheel_thickness / (golden * golden)}" />
   <xacro:property name="platform_radius" value="${0.85 * 0.5 * body_width * golden}" />
@@ -14,4 +18,5 @@
   <xacro:property name="platform_thickness" value="${pole_length * (golden - 1)}" />
   <xacro:property name="pole_radius" value="${platform_thickness * golden}" />
+  <xacro:property name="stem_length" value="${PLATFORM_HEIGHT - body_height - wheel_radius - pole_length}" />
   <!-- Visual turtle elements-->
   <xacro:property name="head_radius" value="${body_width * (golden - 1)/2}" />
@@ -128,5 +133,5 @@
   </link>
   <joint name="tip" type="revolute">
-    <origin xyz="0 0 ${pole_length/2 + platform_thickness/2}" rpy="0 0 0" />
+    <origin xyz="0 0 ${pole_length/2 + platform_thickness}" rpy="0 0 0" />
     <axis xyz="0 1 0"/>
     <limit lower="${-0.187}" upper="${0.187}" effort="100.0" velocity="100.0"/>
